File: Kicad/electronics_tx_p16.sch (KiCad schematic (older format))
At the start: 29 parts

Commit message: rapport diapo
Parts:
- removed K?: CONN_3, symbol CONN_3
- removed P?: CONN_2, symbol CONN_2
- added P?: CONN_7, symbol CONN_7
- added P?: CONN_6, symbol CONN_6
- added Q? (x3): BC547, TO92, symbol BC547
- added R? (x3): 1k, ~, symbol R
- added R? (x2): 47k, ~, symbol R
- added R? (x2): 10k, ~, symbol R
- gave numbers to parts that had none: 27
Connections:
- net labels added: +24VDC_Asynchrone, Capteur_+_Force, Capteur_-_Force, Commande Asynchrone, Curent_limit_Brushless, Dir_Brushless, Dir_output_Brushless, Encoder_Output_Brushless, Foward_asynchrone, On/Off_Brushless, Redemarage_asynchrone, Reset_Asynchrone, Reverse_Asynchrone, Sens_Capteur_Force, Sens_antihoraire_asynchrone, Sens_horaire_asynchrone
- net labels removed: Capteur_+, Capteur_-, Capteur_Brushless, Sens_Capteur
- wire segments 83 -> 119
Other:
- moved on the sheet: C1, C2, C3, R1, R10, R2, R9, RV2, U1A
